File: hardware/amiga_drawbridge_adapter.kicad_sch (KiCad schematic)
At the start: 17 parts, among them J1 FTDI_232_RED, J2 DiskDrive Power, J3 PC3-PC5, J4 AVR-ISP-6, J5 DiskDrive Data, SW1 SW_Push, U1 ATmega328P-A, Y1 16MHz

Commit message: create gerberfiles rev1.0
Parts:
- R1: value 82 -> 100
Changed lines of the file:
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@@
     (in_bom yes) (on_board yes)
     (property "Reference" "R1" (id 0) (at 46.99 166.37 90))
-    (property "Value" "82" (id 1) (at 46.99 173.99 90))
+    (property "Value" "100" (id 1) (at 46.99 173.99 90))
     (property "Footprint" "Resistor_SMD:R_0805_2012Metric_Pad1.20x1.40mm_HandSolder" (id 2) (at 46.99 171.958 90)
       (effects (font (size 1.27 1.27)) hide)
@@
     )
     (path "/c32a7a09-f6b5-4f42-b95d-1874d2997e18"
-      (reference "R1") (unit 1) (value "82") (footprint "Resistor_SMD:R_0805_2012Metric_Pad1.20x1.40mm_HandSolder")
+      (reference "R1") (unit 1) (value "100") (footprint "Resistor_SMD:R_0805_2012Metric_Pad1.20x1.40mm_HandSolder")
     )
     (path "/619a1e7a-12d6-471e-95fb-51051cca37bb"
